Commit message: jazzy-devel

File: models/rbsummit/rbsummit.urdf (robot description, URDF)
Before this commit: robot summit_xl, 22 links, 21 joints
Links:
- link base_link: geometry collision mesh filename=package://robotnik_mujoco/models/rbsummit/rbsummit_xl_chass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; visual mesh filename=package://robotnik_mujoco/models/rbsummit/rbsummit_xl_chass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
- link front_rgbd_camera_link: geometry collision box size=0.02505 0.09 0.025; visual mesh filename=package://robotnik_mujoco/models/rbsummit/intel_d435.stl
- link gps_base_link: geometry collision mesh filename=package://robotnik_mujoco/models/rbsummit/antenna_ANN_MB.stl scale=1.0 1.0 1.0; visual mesh filename=package://robotnik_mujoco/models/rbsummit/antenna_ANN_MB.stl scale=1.0 1.0 1.0
- link gps_mast_base_link: geometry collision mesh filename=package://robotnik_mujoco/models/rbsummit/mastil_gps.stl scale=1.0 1.0 1.0; visual mesh filename=package://robotnik_mujoco/models/rbsummit/mastil_gps.stl scale=1.0 1.0 1.0
- link imu_base_link: geometry collision box size=0.036 0.037 0.009; visual mesh filename=package://robotnik_mujoco/models/rbsummit/vectornav_vn100.s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
- link robot_back_left_wheel: geometry collision mesh filename=package://robotnik_mujoco/models/rbsummit/rubber_wheel.stl; visual mesh filename=package://robotnik_mujoco/models/rbsummit/rubber_wheel.stl
- link robot_back_right_wheel: geometry collision mesh filename=package://robotnik_mujoco/models/rbsummit/rubber_wheel.stl; visual mesh filename=package://robotnik_mujoco/models/rbsummit/rubber_wheel.stl
- link robot_front_left_wheel: geometry collision mesh filename=package://robotnik_mujoco/models/rbsummit/rubber_wheel.stl; visual mesh filename=package://robotnik_mujoco/models/rbsummit/rubber_wheel.stl
- link robot_front_right_wheel: geometry collision mesh filename=package://robotnik_mujoco/models/rbsummit/rubber_wheel.stl; visual mesh filename=package://robotnik_mujoco/models/rbsummit/rubber_wheel.stl
- link top_3d_laser_base_link: geometry collision mesh filename=package://robotnik_mujoco/models/rbsummit/helios_16p.stl; visual mesh filename=package://robotnik_mujoco/models/rbsummit/helios_16p.stl

File: models/rbwatcher/rbwatcher.urdf (robot description, URDF)
Before this commit: robot rbwatcher, 30 links, 29 joints
Links:
- link robot_back_left_wheel: geometry collision mesh filename=package://robotnik_mujoco/models/rbwatcher/rubber_wheel.stl; visual mesh filename=package://robotnik_mujoco/models/rbwatcher/rubber_wheel.stl
- link robot_back_right_wheel: geometry collision mesh filename=package://robotnik_mujoco/models/rbwatcher/rubber_wheel.stl; visual mesh filename=package://robotnik_mujoco/models/rbwatcher/rubber_wheel.stl
- link robot_base_link: geometry collision mesh filename=package://robotnik_mujoco/models/rbwatcher/rbwatcher_chassi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; visual mesh filename=package://robotnik_mujoco/models/rbwatcher/rbwatcher_chassi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
- link robot_front_left_wheel: geometry collision mesh filename=package://robotnik_mujoco/models/rbwatcher/rubber_wheel.stl; visual mesh filename=package://robotnik_mujoco/models/rbwatcher/rubber_wheel.stl
- link robot_front_rgbd_camera_link: geometry collision box size=0.02505 0.09 0.025; visual mesh filename=package://robotnik_mujoco/models/rbwatcher/intel_d435_color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
- link robot_front_right_wheel: geometry collision mesh filename=package://robotnik_mujoco/models/rbwatcher/rubber_wheel.stl; visual mesh filename=package://robotnik_mujoco/models/rbwatcher/rubber_wheel.stl
- link robot_imu_base_link: geometry collision box size=0.036 0.037 0.009; visual mesh filename=package://robotnik_mujoco/models/rbwatcher/vectornav_vn100.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
- link robot_top_3d_laser_base_link: geometry collision mesh filename=package://robotnik_mujoco/models/rbwatcher/helios_16p.stl; visual mesh filename=package://robotnik_mujoco/models/rbwatcher/helios_16p.stl
- link robot_top_ptz_camera_base_link: geometry collision mesh filename=package://robotnik_mujoco/models/rbwatcher/link_750_base.stl scale=0.001 0.001 0.001; visual mesh filename=package://robotnik_mujoco/models/rbwatcher/link_750_base.stl scale=0.001 0.001 0.001
- link robot_top_ptz_camera_pan_link: geometry collision mesh filename=package://robotnik_mujoco/models/rbwatcher/link_750_pan.stl scale=1.0 1.0 1.0; visual mesh filename=package://robotnik_mujoco/models/rbwatcher/link_750_pan.stl scale=1.0 1.0 1.0
- link robot_top_ptz_camera_tilt_link: geometry collision mesh filename=package://robotnik_mujoco/models/rbwatcher/link_750_tilt.stl scale=1.0 1.0 1.0; visual mesh filename=package://robotnik_mujoco/models/rbwatcher/link_750_tilt.stl scale=1.0 1.0 1.0
- link robot_top_structure_link: geometry collision mesh filename=package://robotnik_mujoco/models/rbwatcher/rbwatcher_top_st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; visual mesh filename=package://robotnik_mujoco/models/rbwatcher/rbwatcher_top_st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
